Commit message: feat: Introduce dynamixel_hardware_interface_example_1 package for dual ros2_control setup

File: dynamixel_hardware_interface_example/config/dynamixel_system.urdf.xacro (robot description, xacro)
@@ -2,6 +2,8 @@
 <robot xmlns:xacro="http://www.ros.org/wiki/xacro" name="dynamixel_system">
   <xacro:arg name="prefix" default="" />
+  <xacro:arg name="baud_rate" default="4000000" />
+  <xacro:arg name="port_name" default="/dev/ttyUSB0" />
   <xacro:include filename="dynamixel_system.ros2_control.xacro" />
-  <xacro:dynamixel_system_ros2_control name="dynamixel_system"/>
+  <xacro:dynamixel_system_ros2_control name="dynamixel_system" port_name="$(arg port_name)" baud_rate="$(arg baud_rate)"/>
   <link name="$(arg prefix)base_link"/>
   <joint name="$(arg prefix)joint1" type="revolute">

File: dynamixel_hardware_interface_example_1/config/dynamixel_system_1.ros2_control.xacro (robot description, xacro)
@@ -1,6 +1,6 @@
 <?xml version="1.0"?>
 <robot xmlns:xacro="http://www.ros.org/wiki/xacro">
-  <xacro:macro name="dynamixel_system_ros2_control" params="name port_name baud_rate">
-    <ros2_control name="${name}" type="system">
+  <xacro:macro name="dynamixel_system_ros2_control_1" params="name port_name baud_rate">
+    <ros2_control name="${name}" type="system" is_async="true">
       <hardware>
         <plugin>dynamixel_hardware_interface/DynamixelHardware</plugin>

File: dynamixel_hardware_interface_example_1/config/dynamixel_system_2.ros2_control.xacro (robot description, xacro)
@@ -1,6 +1,6 @@
 <?xml version="1.0"?>
 <robot xmlns:xacro="http://www.ros.org/wiki/xacro">
-  <xacro:macro name="dynamixel_system_ros2_control" params="name port_name baud_rate">
-    <ros2_control name="${name}" type="system">
+  <xacro:macro name="dynamixel_system_ros2_control_2" params="name port_name baud_rate">
+    <ros2_control name="${name}" type="system" is_async="true">
       <hardware>
         <plugin>dynamixel_hardware_interface/DynamixelHardware</plugin>
@@ -24,12 +24,12 @@
         <param name="set_dxl_torque_srv_name">dynamixel_hardware_interface/set_dxl_torque</param>
       </hardware>
-      <joint name="joint1">
+      <joint name="joint2">
         <command_interface name="position"/>
         <state_interface name="position"/>
         <state_interface name="velocity"/>
       </joint>
-      <gpio name="dxl1">
+      <gpio name="dxl2">
         <param name="type">dxl</param>
-        <param name="ID">1</param>
+        <param name="ID">2</param>
         <command_interface name="Goal Position"/>
         <state_interface name="Present Position"/>
